Commit message: update from last night

File: dynamixel_arm/urdf/acps.urdf (robot description, URDF)
Before this commit: robot acps, 5 links, 4 joints
Links:
- link base_link: geometry collision mesh filename=package://dynamixel_arm/meshes/base_link.STL; visual mesh filename=package://dynamixel_arm/meshes/base_link.STL
- link link1: geometry collision mesh filename=package://dynamixel_arm/meshes/link1.STL; visual mesh filename=package://dynamixel_arm/meshes/link1.STL
- link link2: geometry collision mesh filename=package://dynamixel_arm/meshes/link2.STL; visual mesh filename=package://dynamixel_arm/meshes/link2.STL
- link link3: geometry collision mesh filename=package://dynamixel_arm/meshes/link3.STL; visual mesh filename=package://dynamixel_arm/meshes/link3.STL
- link link4: geometry collision mesh filename=package://dynamixel_arm/meshes/link4.STL; visual mesh filename=package://dynamixel_arm/meshes/link4.STL

Commit message: setup gazebo

File: dynamixel_arm/urdf/acps.urdf (robot description, URDF)
Before this commit: robot acps, 5 links, 4 joints
Links:
- link base_link: mass 0.043005 -> 0.090196
- link link1: mass 0.053822 -> 0.05394
- link link2: mass 0.055878 -> 0.080328
- link link3: mass 0.055878 -> 0.080328
- link link4: mass 0.012873 -> 0.011748
Joints:
- removed joint theta1
- removed joint theta2
- removed joint theta3
- removed joint theta4
- added joint joint1: type continuous, parent base_link, child link1, origin xyz=0 0 0.0548 rpy=0 0 0, axis 0 0 1
- added joint joint2: type continuous, parent link1, child link2, origin xyz=0 0 0.04355 rpy=1.5708 0 0, axis 0 0 -1
- added joint joint3: type continuous, parent link2, child link3, origin xyz=0.11855 0 0 rpy=0 0 0, axis 0 0 -1
- added joint joint4: type continuous, parent link3, child link4, origin xyz=0.11855 0 0 rpy=0 0 0, axis 0 0 -1
