Commit message: fixing gazebo

File: dynamixel_arm/urdf/acps_bot.ros2_control_gazebo.xacro (robot description, xacro)
@@ -37,5 +37,5 @@
     <gazebo>
       <plugin filename="libign_ros2_control-system.so" name="ign_ros2_control::IgnitionROS2ControlPlugin">
-        <parameters>$(find acps_bot_description)/controllers/controllers.yaml</parameters>
+        <parameters>$(find dynamixel_arm)/controllers/controllers.yaml</parameters>
       </plugin>
     </gazebo>

File: dynamixel_arm/urdf/acps_bot.urdf.xacro (robot description, xacro)
@@ -1,10 +1,10 @@
 <?xml version="1.0"?>
 <robot name="acps_bot" xmlns:xacro="http://ros.org/wiki/xacro">
-  <xacro:include filename="$(find acps_bot_description)/urdf/acps_bot.xacro" />
-  <xacro:include filename="$(find acps_bot_description)/urdf/acps_bot.ros2_control_gazebo.xacro" />
+  <xacro:include filename="$(find dynamixel_arm)/urdf/acps_bot.xacro" />
+  <xacro:include filename="$(find dynamixel_arm)/urdf/acps_bot.ros2_control_gazebo.xacro" />
   <link name="world"/>
   <xacro:acps_bot parent="world">
     <origin xyz="0 0 0" rpy="0 0 0" />
-  </xacro:pantilt_bot>
+  </xacro:acps_bot>
   <xacro:acps_bot_ros2_control name="acps_bot_ros2_control" />
 </robot>

File: dynamixel_arm/urdf/acps_bot.xacro (robot description, xacro)
@@ -82,17 +82,4 @@
         </collision>
     </link>
-    <joint
-        name="joint1"
-        type="continuous">
-        <origin
-        xyz="0 0 0.0548"
-        rpy="0 0 0" />
-        <parent
-        link="base_link" />
-        <child
-        link="link1" />
-        <axis
-        xyz="0 0 1" />
-    </joint>
     <link
         name="link2">
@@ -135,17 +122,4 @@
         </collision>
     </link>
-    <joint
-        name="joint2"
-        type="continuous">
-        <origin
-        xyz="0 0 0.04355"
-        rpy="1.5708 0 0" />
-        <parent
-        link="link1" />
-        <child
-        link="link2" />
-        <axis
-        xyz="0 0 -1" />
-    </joint>
     <link
         name="link3">
@@ -188,17 +162,4 @@
         </collision>
     </link>
-    <joint
-        name="joint3"
-        type="continuous">
-        <origin
-        xyz="0.11855 0 0"
-        rpy="0 0 0" />
-        <parent
-        link="link2" />
-        <child
-        link="link3" />
-        <axis
-        xyz="0 0 -1" />
-    </joint>
     <link
         name="link4">
@@ -241,6 +202,37 @@
         </collision>
     </link>
-    <joint
-        name="joint4"
+    <joint name="origin_to_joint1" type="fixed">
+      <xacro:insert_block name="origin" />
+      <parent link="${parent}" />
+      <child link="base_link" />
+    </joint>
+    <joint
+        name="joint1"
+        type="continuous">
+        <origin
+        xyz="0 0 0.0548"
+        rpy="0 0 0" />
+        <parent
+        link="base_link" />
+        <child
+        link="link1" />
+        <axis
+        xyz="0 0 1" />
+    </joint>
+    <joint
+        name="joint2"
+        type="continuous">
+        <origin
+        xyz="0 0 0.04355"
+        rpy="1.5708 0 0" />
+        <parent
+        link="link1" />
+        <child
+        link="link2" />
+        <axis
+        xyz="0 0 -1" />
+    </joint>
+    <joint
+        name="joint3"
         type="continuous">
         <origin
@@ -248,4 +240,17 @@
         rpy="0 0 0" />
         <parent
+        link="link2" />
+        <child
+        link="link3" />
+        <axis
+        xyz="0 0 -1" />
+    </joint>
+    <joint
+        name="joint4"
+        type="continuous">
+        <origin
+        xyz="0.11855 0 0"
+        rpy="0 0 0" />
+        <parent
         link="link3" />
         <child
