Commit message: gazebo and interface

File: dynamixel_arm/urdf/acps_bot.ros2_control.xacro (robot description, xacro)
@@ -3,9 +3,10 @@
   <xacro:macro name="acps_bot_ros2_control" params="name">
     <ros2_control name="${name}" type="system">
-      <!-- <hardware>
+      <hardware>
         <plugin>dynamixel_hardware/DynamixelHardware</plugin>
         <param name="usb_port">/dev/ttyUSB0</param>
         <param name="baud_rate">1000000</param>
-      </hardware> -->
+        <!-- <param name="use_dummy">true</param> -->
+      </hardware>
       <joint name="joint1">
         <param name="id">11</param>
@@ -24,20 +25,4 @@
         <state_interface name="effort"/>
       </joint>
-      <joint name="joint3">
-        <param name="id">13</param>
-        <command_interface name="position"/>
-        <command_interface name="velocity"/>
-        <state_interface name="position"/>
-        <state_interface name="velocity"/>
-        <state_interface name="effort"/>
-      </joint>
-      <joint name="joint4">
-        <param name="id">14</param>
-        <command_interface name="position"/>
-        <command_interface name="velocity"/>
-        <state_interface name="position"/>
-        <state_interface name="velocity"/>
-        <state_interface name="effort"/>
-      </joint>
     </ros2_control>
   </xacro:macro>

File: dynamixel_arm/urdf/acps_bot.ros2_control_gazebo.xacro (robot description, xacro)
@@ -1,5 +1,5 @@
 <?xml version="1.0"?>
 <robot xmlns:xacro="http://www.ros.org/wiki/xacro">
-  <xacro:macro name="acps_bot_ros2_control" params="name">
+  <xacro:macro name="acps_bot_ros2_control_gazebo" params="name">
     <ros2_control name="${name}" type="system">
       <hardware>
@@ -35,9 +35,9 @@
       </joint>
     </ros2_control>
-    <gazebo>
-      <plugin name="ign_ros2_control::IgnitionROS2ControlPlugin" filename="libign_ros2_control-system.so">
-        <parameters>$(find dynamixel_arm)/controllers/controllers.yaml</parameters>
-      </plugin>
-    </gazebo>
+  <gazebo>
+    <plugin filename="ign_ros2_control-system" name="ign_ros2_control::IgnitionROS2ControlPlugin">
+      <parameters>$(find dynamixel_arm)/config/acps_controller.yaml</parameters>
+    </plugin>
+  </gazebo>
   </xacro:macro>
 </robot>

File: dynamixel_arm/urdf/acps_bot.urdf.xacro (robot description, xacro)
@@ -3,8 +3,6 @@
   <xacro:include filename="$(find dynamixel_arm)/urdf/acps_bot.xacro" />
   <xacro:include filename="$(find dynamixel_arm)/urdf/acps_bot.ros2_control_gazebo.xacro" />
-  <link name="world"/>
-  <xacro:acps_bot parent="world">
-    <origin xyz="0 0 0" rpy="0 0 0" />
-  </xacro:acps_bot>
-  <xacro:acps_bot_ros2_control name="acps_bot_ros2_control" />
+  <!-- <link name="world"/> -->
+  <xacro:acps_bot/>
+  <xacro:acps_bot_ros2_control_gazebo name="acps_bot_ros2_control_gazebo" />
 </robot>

File: dynamixel_arm/urdf/acps_bot.xacro (robot description, xacro)
@@ -1,5 +1,6 @@
 <?xml version="1.0"?>
-<robot xmlns:xacro="http://ros.org/wiki/xacro">
-    <xacro:macro name="acps_bot" params="parent *origin">
+<robot xmlns:xacro="http://www.ros.org/wiki/xacro">
+<xacro:macro name="acps_bot">
+    <link name="world"/>
     <link
         name="base_link">
@@ -203,7 +204,7 @@
     </link>
     <joint name="origin_to_joint1" type="fixed">
-      <xacro:insert_block name="origin" />
-      <parent link="${parent}" />
-      <child link="base_link" />
+        <origin rpy="0 0 0" xyz="0 0 0"/>
+        <parent link="world"/>
+        <child link="base_link"/>
     </joint>
     <joint
